Commit message: camera on model

File: catkin_ws/src/simple_hexapod_description/urdf/simple_hexapod.xacro (robot description, xacro)
@@ -517,5 +517,5 @@
 </joint>
 <!-- Camera -->
-<link name="camera_link">
+<!-- <link name="camera_link">
   <collision>
     <origin xyz="0 0 0" rpy="0 0 0"/>
@@ -535,10 +535,14 @@
     <inertia ixx="1e-6" ixy="0" ixz="0" iyy="1e-6" iyz="0" izz="1e-6" />
   </inertial>
-</link>
-<joint name="camera_joint" type="fixed">
+</link> -->
+<!-- <joint name="camera_joint" type="fixed">
   <axis xyz="0 1 0" />
   <origin xyz="0.06 0 0.2" rpy="0 0 0"/>
   <parent link="base_link"/>
   <child link="camera_link"/>
-</joint>
+</joint> -->
+<xacro:include filename="$(find realsense2_description)/urdf/_d435.urdf.xacro" />
+<xacro:sensor_d435 name="camera" topics_ns="camera" parent="base_link" publish_pointcloud="true">
+  <origin xyz="0 0 0.3" rpy="0 0.6981 0" />
+</xacro:sensor_d435>
 </robot>

Commit message: 13 july

File: catkin_ws/src/simple_hexapod_description/urdf/simple_hexapod.xacro (robot description, xacro)
@@ -542,7 +542,7 @@
   <child link="camera_link"/>
 </joint> -->
-<xacro:include filename="$(find realsense2_description2)/urdf/_d435.urdf.xacro" />
+<xacro:include filename="$(find realsense2_description)/urdf/_d435.urdf.xacro" />
 <xacro:sensor_d435 name="camera" topics_ns="camera" parent="base_link" publish_pointcloud="true">
-  <origin xyz="0 0 0.3" rpy="0 0.6981 0" />
+  <origin xyz="0.055 0 0.15" rpy="0 0.5236 0" />
 </xacro:sensor_d435>
 </robot>

Commit message: 21 julie

File: catkin_ws/src/simple_hexapod_description/urdf/simple_hexapod.xacro (robot description, xacro)
@@ -544,5 +544,5 @@
 <xacro:include filename="$(find realsense2_description)/urdf/_d435.urdf.xacro" />
 <xacro:sensor_d435 name="camera" topics_ns="camera" parent="base_link" publish_pointcloud="true">
-  <origin xyz="0.055 0 0.15" rpy="0 0.5236 0" />
+  <origin xyz="0.055 0 0.13" rpy="0 0.5236 0" />
 </xacro:sensor_d435>
 </robot>

Commit message: update 26aug

File: catkin_ws/src/simple_hexapod_description/urdf/simple_hexapod.xacro (robot description, xacro)
@@ -544,5 +544,5 @@
 <xacro:include filename="$(find realsense2_description)/urdf/_d435.urdf.xacro" />
 <xacro:sensor_d435 name="camera" topics_ns="camera" parent="base_link" publish_pointcloud="true">
-  <origin xyz="0.055 0 0.13" rpy="0 0.5236 0" />
+  <origin xyz="0.017 0 0.210" rpy="0 0.6109 0" />
 </xacro:sensor_d435>
 </robot>
